File: HardWare/AutonomousSensorBoard V1.sch (EAGLE design)
At the start: 10 parts

Commit message: gerbers generated
Parts:
- added FRAME1: FRAME-LEDGER, SparkFun-Aesthetics:FRAME-LEDGER
- added H1, H2, H3, H4: STAND-OFF, SparkFun-Electromechanical:STAND-OFF
- added J1, J2, J3, J4, J5: (no value), SparkFun-Connectors:M03LOCK
Connections:
- new net A0: J1.3, U$1.A0
- new net A1: J2.3, U$1.A1
- new net A2: J3.3, U$1.A2
- new net A3: J4.3, U$1.A3
- new net A4: J5.3, U$1.A4
- net 3.3V: now also J1.2, J2.2, J3.2, J4.2, J5.2
- net GND: now also J1.1, J2.1, J3.1, J4.1, J5.1
